File: K3NG-rotator-shield.kicad_pcb (KiCad board)
At the start: 2 copper layers, 59.2 x 135.6 mm, 18 parts, among them J14 Conn_01x01_Pin, J15 Conn_01x01_Pin, J2 Conn_01x04_Socket, J3 Conn_01x02_Pin, J4 Conn_01x04_Socket, J6 Conn_01x07_Socket, J7 Conn_01x06_Socket, U1 DRV8251ADDAR, U2 DRV8251ADDAR

Commit message: Add files via upload
Routing:
- net RotateDown-OUT: track 14.5 -> 13.6 mm
Changed lines of the file:
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@@
 	)
 	(gr_text "THERMAL PASTE AREA"
-		(at 148.6 150.4 0)
+		(at 148.6 150 0)
 		(layer "F.SilkS")
 		(effects
@@
 	)
 	(segment
+		(start 134.25 80.86)
+		(end 131.7 83.41)
+		(width 0.6)
+		(layer "B.Cu")
+		(net 3)
+	)
+	(segment
+		(start 131.7 83.41)
+		(end 131.7 123.1)
+		(width 0.6)
+		(layer "B.Cu")
+		(net 3)
+	)
+	(segment
+		(start 131.7 123.1)
+		(end 141.568062 132.968062)
+		(width 0.6)
+		(layer "B.Cu")
+		(net 3)
+	)
+	(segment
+		(start 148 136.5)
+		(end 153.1998 141.6998)
+		(width 0.6)
+		(layer "B.Cu")
+		(net 3)
+	)
+	(segment
+		(start 153.1998 141.6998)
+		(end 169.2684 141.6998)
+		(width 0.6)
+		(layer "B.Cu")
+		(net 3)
+	)
+	(segment
+		(start 141.79 132.968062)
+		(end 145.321938 136.5)
+		(width 0.6)
+		(layer "B.Cu")
+		(net 3)
+	)
+	(segment
 		(start 145.321938 136.5)
 		(end 148 136.5)
@@
 	)
 	(segment
-		(start 148 136.5)
-		(end 153.1998 141.6998)
-		(width 0.6)
-		(layer "B.Cu")
-		(net 3)
-	)
-	(segment
-		(start 141.79 132.968062)
-		(end 145.321938 136.5)
-		(width 0.6)
-		(layer "B.Cu")
-		(net 3)
-	)
-	(segment
-		(start 131.939 122.739)
-		(end 141.79 132.59)
-		(width 0.6)
-		(layer "B.Cu")
-		(net 3)
-	)
-	(segment
-		(start 153.1998 141.6998)
-		(end 169.2684 141.6998)
-		(width 0.6)
-		(layer "B.Cu")
-		(net 3)
-	)
-	(segment
-		(start 141.79 132.59)
+		(start 141.568062 132.968062)
 		(end 141.79 132.968062)
-		(width 0.6)
-		(layer "B.Cu")
-		(net 3)
-	)
-	(segment
-		(start 131.939 83.171)
-		(end 131.939 122.739)
-		(width 0.6)
-		(layer "B.Cu")
-		(net 3)
-	)
-	(segment
-		(start 134.25 80.86)
-		(end 131.939 83.171)
 		(width 0.6)
 		(layer "B.Cu")
@@
 	)
 	(segment
+		(start 180.5788 125.5797)
+		(end 173.2075 132.951)
+		(width 0.6)
+		(layer "F.Cu")
+		(net 6)
+	)
+	(segment
+		(start 166.6264 140.8894)
+		(end 166.6264 144.8559)
+		(width 0.6)
+		(layer "F.Cu")
+		(net 6)
+	)
+	(segment
+		(start 168.2405 146.47)
+		(end 168.8 146.47)
+		(width 0.6)
+		(layer "F.Cu")
+		(net 6)
+	)
+	(segment
+		(start 166.6264 144.8559)
+		(end 168.2405 146.47)
+		(width 0.6)
+		(layer "F.Cu")
+		(net 6)
+	)
+	(segment
+		(start 173.2075 134.3083)
+		(end 166.6264 140.8894)
+		(width 0.6)
+		(layer "F.Cu")
+		(net 6)
+	)
+	(segment
 		(start 173.2075 132.951)
 		(end 173.2075 134.3083)
-		(width 0.6)
-		(layer "F.Cu")
-		(net 6)
-	)
-	(segment
-		(start 173.2075 134.3083)
-		(end 166.6264 140.8894)
-		(width 0.6)
-		(layer "F.Cu")
-		(net 6)
-	)
-	(segment
-		(start 166.6264 140.8894)
-		(end 166.6264 144.8559)
-		(width 0.6)
-		(layer "F.Cu")
-		(net 6)
-	)
-	(segment
-		(start 168.2405 146.47)
-		(end 168.8 146.47)
-		(width 0.6)
-		(layer "F.Cu")
-		(net 6)
-	)
-	(segment
-		(start 166.6264 144.8559)
-		(end 168.2405 146.47)
-		(width 0.6)
-		(layer "F.Cu")
-		(net 6)
-	)
-	(segment
-		(start 180.5788 125.5797)
-		(end 173.2075 132.951)
 		(width 0.6)
 		(layer "F.Cu")
@@
 	(segment
 		(start 184.8254 70.415)
+		(end 182.51 68.0996)
+		(width 0.6)
+		(layer "B.Cu")
+		(net 6)
+	)
+	(segment
+		(start 182.51 68.0996)
+		(end 182.51 66.636)
+		(width 0.6)
+		(layer "B.Cu")
+		(net 6)
+	)
+	(segment
+		(start 180.5788 125.5797)
 		(end 184.8254 121.3331)
 		(width 0.6)
@@
 	)
 	(segment
-		(start 182.51 66.636)
-		(end 182.51 68.0996)
-		(width 0.6)
-		(layer "B.Cu")
-		(net 6)
-	)
-	(segment
-		(start 182.51 68.0996)
+		(start 184.8254 121.3331)
 		(end 184.8254 70.415)
-		(width 0.6)
-		(layer "B.Cu")
-		(net 6)
-	)
-	(segment
-		(start 184.8254 121.3331)
-		(end 180.5788 125.5797)
 		(width 0.6)
 		(layer "B.Cu")
@@
 	)
 	(segment
+		(start 131.8 123.7718)
+		(end 136.1857 128.1575)
+		(width 0.6)
+		(layer "F.Cu")
+		(net 9)
+	)
+	(segment
 		(start 136.1857 128.1575)
 		(end 136.1857 140.5853)
@@
 	)
 	(segment
+		(start 143.3404 147.74)
+		(end 143.88 147.74)
+		(width 0.6)
+		(layer "F.Cu")
+		(net 9)
+	)
+	(segment
 		(start 168.2146 147.74)
 		(end 168.8 147.74)
@@
 	)
 	(segment
-		(start 134.25 60.54)
-		(end 131.939 62.851)
-		(width 0.6)
-		(layer "F.Cu")
-		(net 9)
-	)
-	(segment
-		(start 131.939 62.851)
-		(end 131.939 123.9108)
+		(start 136.1857 140.5853)
+		(end 143.3404 147.74)
 		(width 0.6)
 		(layer "F.Cu")
@@
 	)
 	(segment
-		(start 143.3404 147.74)
-		(end 143.88 147.74)
-		(width 0.6)
-		(layer "F.Cu")
-		(net 9)
-	)
-	(segment
-		(start 131.939 123.9108)
-		(end 136.1857 128.1575)
-		(width 0.6)
-		(layer "F.Cu")
-		(net 9)
-	)
-	(segment
-		(start 136.1857 140.5853)
-		(end 143.3404 147.74)
+		(start 134.25 60.54)
+		(end 131.8 62.99)
+		(width 0.6)
+		(layer "F.Cu")
+		(net 9)
+	)
+	(segment
+		(start 131.8 62.99)
+		(end 131.8 123.7718)
 		(width 0.6)
 		(layer "F.Cu")
@@
 	)
 	(segment
-		(start 185.8 140.4)
-		(end 183.65 140.4)
+		(start 175.34 142.34)
+		(end 177.6906 139.9894)
 		(width 2)
 		(layer "F.Cu")
@@
 	)
 	(segment
-		(start 183.65 140.4)
-		(end 183.2394 139.9894)
-		(width 2)
-		(layer "F.Cu")
-		(net 15)
-	)
-	(segment
-		(start 183.2394 139.9894)
-		(end 177.6906 139.9894)
-		(width 2)
-		(layer "F.Cu")
-		(net 15)
-	)
-	(segment
-		(start 177.6906 139.9894)
+		(start 175.34 142.34)
 		(end 173.75 143.93)
 		(width 0.601)
@@
 	)
 	(segment
-		(start 151.0728 143.1331)
+		(start 183.2394 139.9894)
+		(end 183.65 140.4)
+		(width 2)
+		(layer "F.Cu")
+		(net 15)
+	)
+	(segment
+		(start 183.65 140.4)
+		(end 185.8 140.4)
+		(width 2)
+		(layer "F.Cu")
+		(net 15)
+	)
+	(segment
+		(start 177.6906 139.9894)
+		(end 183.2394 139.9894)
+		(width 2)
+		(layer "F.Cu")
+		(net 15)
+	)
+	(segment
+		(start 162 143.1331)
 		(end 149.6269 143.1331)
 		(width 2)
@@
 	)
 	(via
-		(at 151.0728 143.1331)
+		(at 162 143.1331)
 		(size 0.6)
 		(drill 0.3)
@@
 	)
 	(segment
-		(start 151.0728 143.1331)
-		(end 172.7466 143.1331)
-		(width 2)
-		(layer "B.Cu")
-		(net 16)
-	)
-	(segment
 		(start 175.0935 145.48)
 		(end 185.8 145.48)
@@
 		(layer "B.Cu")
 		(net 16)
+	)
+	(segment
+		(start 162 143.1331)
+		(end 172.7466 143.1331)
+		(width 2)
+		(layer "B.Cu")
+		(net 16)
+	)
+	(segment
+		(start 179.7795 142.94)
+		(end 185.8 142.94)
+		(width 2)
+		(layer "F.Cu")
+		(net 17)
+	)
+	(segment
+		(start 176.2 146.5195)
+		(end 179.7795 142.94)
+		(width 2)
+		(layer "F.Cu")
+		(net 17)
 	)
 	(segment
@@
 	)
 	(segment
-		(start 181.7302 146.5195)
+		(start 176.2 146.5195)
 		(end 173.7995 146.5195)
 		(width 0.601)
 		(layer "F.Cu")
 		(net 17)
-	)
-	(segment
-		(start 183.65 144.5997)
-		(end 181.7302 146.5195)
-		(width 2)
-		(layer "F.Cu")
-		(net 17)
-	)
-	(segment
-		(start 185.8 142.94)
-		(end 183.65 142.94)
-		(width 2)
-		(layer "F.Cu")
-		(net 17)
-	)
-	(segment
-		(start 183.65 142.94)
-		(end 183.65 144.5997)
-		(width 2)
-		(layer "F.Cu")
-		(net 17)

Commit message: Add files via upload
Parts:
- J3: footprint Connector_PinHeader_2.54mm:PinHeader_1x02_P2.54mm_Vertical -> Connector_Wire:SolderWire-1.5sqmm_1x02_P6mm_D1.7mm_OD3mm
- R1, R2, R3, R4: footprint Resistor_THT:R_Axial_DIN0204_L3.6mm_D1.6mm_P5.08mm_Vertical -> Resistor_THT:R_Axial_DIN0204_L3.6mm_D1.6mm_P5.08mm_Horizontal
- turned J3 to 90 degrees
Routing:
- net GND: vias 3 -> 27
Other:
- board text added: "4A MAX!"
- board text removed: "8A MAX!"
