File: K3NG-rotator-shield.kicad_sch (KiCad schematic)
At the start: 25 parts, among them J1 Conn_01x08_Socket, J10 Conn_01x01_Pin, J11 Conn_01x10_Socket, J12 Conn_01x01_Pin, J13 Conn_01x01_Pin, J14 Conn_01x01_Pin, J15 Conn_01x01_Pin, J2 Conn_01x04_Socket, J3 Conn_01x02_Pin, J4 Conn_01x04_Socket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

Commit message: Add files via upload
Other:
- note added: "ANALOG INPUTS ARDUINO"
- note added: "AREF"
- note added: "D0/RX"
- note added: "D1/TX"
- note added: "D10"
- note added: "D11"
- note added: "D12"
- note added: "D13"
- note added: "D14"
- note added: "D15"
- note added: "D16"
- note added: "D17"
- note added: "D18"
- note added: "D19"
- note added: "D2"
- note added: "D3"
- note added: "D4"
- note added: "D5"
- note added: "D6"
- note added: "D7"
- note added: "D8"
- note added: "D9"
- note added: "GND"
- note added: "SLA"
- note added: "SLC"
- note added: "SWITCHES, ACTIVE IF GROUNDED"
- note removed: "ANALOG"
- note removed: "SWITCHES, ACTIVE ON GROUND"
Changed lines of the file:
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@@
+		)
+	)
+	(text "D1/TX"
+		(exclude_from_sim no)
+		(at 207.772 90.678 0)
+		(effects
+			(font
+				(size 1.27 1.27)
+			)
 		)
 	)
 	(text "I2C and other pins"
 		(exclude_from_sim no)
-		(at 207.772 50.546 90)
+		(at 211.074 50.546 90)
+		(effects
+			(font
+				(size 1.27 1.27)
+			)
+		)
+	)
+	(text "D7"
+		(exclude_from_sim no)
+		(at 205.74 75.184 0)
+		(effects
+			(font
+				(size 1.27 1.27)
+			)
+		)
+	)
+	(text "D15"
+		(exclude_from_sim no)
+		(at 228.346 134.874 0)
+		(effects
+			(font
+				(size 1.27 1.27)
+			)
+		)
+	)
+	(text "D3"
+		(exclude_from_sim no)
+		(at 206.248 85.344 0)
 		(effects
 			(font
@@
 		)
 	)
+	(text "D19"
+		(exclude_from_sim no)
+		(at 228.6 145.288 0)
+		(effects
+			(font
+				(size 1.27 1.27)
+			)
+		)
+	)
+	(text "D14"
+		(exclude_from_sim no)
+		(at 228.346 132.588 0)
+		(effects
+			(font
+				(size 1.27 1.27)
+			)
+		)
+	)
+	(text "D12"
+		(exclude_from_sim no)
+		(at 207.264 52.324 0)
+		(effects
+			(font
+				(size 1.27 1.27)
+			)
+		)
+	)
+	(text "D5"
+		(exclude_from_sim no)
+		(at 205.74 80.518 0)
+		(effects
+			(font
+				(size 1.27 1.27)
+			)
+		)
+	)
 	(text "GPIO "
 		(exclude_from_sim no)
-		(at 208.026 82.804 90)
+		(at 211.582 82.804 90)
+		(effects
+			(font
+				(size 1.27 1.27)
+			)
+		)
+	)
+	(text "D18"
+		(exclude_from_sim no)
+		(at 228.6 142.748 0)
 		(effects
 			(font
@@
 		)
 	)
-	(text "   SWITCHES,\nACTIVE ON GROUND"
+	(text "D16"
+		(exclude_from_sim no)
+		(at 228.346 137.414 0)
+		(effects
+			(font
+				(size 1.27 1.27)
+			)
+		)
+	)
+	(text "D9"
+		(exclude_from_sim no)
+		(at 206.248 59.944 0)
+		(effects
+			(font
+				(size 1.27 1.27)
+			)
+		)
+	)
+	(text "   SWITCHES,\nACTIVE IF GROUNDED"
 		(exclude_from_sim no)
 		(at 164.338 85.598 90)
@@
 		)
 	)
-	(text "ANALOG"
-		(exclude_from_sim no)
-		(at 228.6 138.176 90)
+	(text "D10"
+		(exclude_from_sim no)
+		(at 206.756 57.404 0)
+		(effects
+			(font
+				(size 1.27 1.27)
+			)
+		)
+	)
+	(text "ANALOG INPUTS\nARDUINO"
+		(exclude_from_sim no)
+		(at 233.426 138.176 90)
+		(effects
+			(font
+				(size 1.27 1.27)
+			)
+		)
+	)
+	(text "SLC"
+		(exclude_from_sim no)
+		(at 207.01 39.624 0)
 		(effects
 			(font
@@
 		)
 	)
+	(text "D0/RX"
+		(exclude_from_sim no)
+		(at 208.026 92.964 0)
+		(effects
+			(font
+				(size 1.27 1.27)
+			)
+		)
+	)
+	(text "D13"
+		(exclude_from_sim no)
+		(at 207.01 49.784 0)
+		(effects
+			(font
+				(size 1.27 1.27)
+			)
+		)
+	)
+	(text "D6"
+		(exclude_from_sim no)
+		(at 205.994 77.724 0)
+		(effects
+			(font
+				(size 1.27 1.27)
+			)
+		)
+	)
+	(text "D17"
+		(exclude_from_sim no)
+		(at 228.346 140.208 0)
+		(effects
+			(font
+				(size 1.27 1.27)
+			)
+		)
+	)
+	(text "D4"
+		(exclude_from_sim no)
+		(at 205.994 82.804 0)
+		(effects
+			(font
+				(size 1.27 1.27)
+			)
+		)
+	)
+	(text "D11"
+		(exclude_from_sim no)
+		(at 207.01 54.864 0)
+		(effects
+			(font
+				(size 1.27 1.27)
+			)
+		)
+	)
+	(text "SLA"
+		(exclude_from_sim no)
+		(at 207.01 42.164 0)
+		(effects
+			(font
+				(size 1.27 1.27)
+			)
+		)
+	)
 	(text "Brushed DC Motor Drivers and related."
 		(exclude_from_sim no)
@@
 		(effects
 			(font
+				(size 1.27 1.27)
+			)
+		)
+	)
+	(text "D8"
+		(exclude_from_sim no)
+		(at 206.248 62.484 0)
+		(effects
+			(font
+				(size 1.27 1.27)
+			)
+		)
+	)
+	(text "GND"
+		(exclude_from_sim no)
+		(at 207.01 47.244 0)
+		(effects
+			(font
+				(size 1.27 1.27)
+			)
+		)
+	)
+	(text "D2"
+		(exclude_from_sim no)
+		(at 206.248 88.138 0)
+		(effects
+			(font
+				(size 1.27 1.27)
+			)
+		)
+	)
+	(text "AREF"
+		(exclude_from_sim no)
+		(at 207.518 44.704 0)
+		(effects
+			(font

Commit message: Add files via upload
Parts:
- removed J1, J8: Conn_01x08_Socket, Connector_PinHeader_2.54mm:PinHeader_1x08_P2.54mm_Vertical, symbol Connector:Conn_01x08_Socket
- removed J10, J12, J13, J5: Conn_01x01_Pin, MountingHole:MountingHole_4.3mm_M4_DIN965_Pad, symbol Connector:Conn_01x01_Pin
- removed J11: Conn_01x10_Socket, Connector_PinHeader_2.54mm:PinHeader_1x10_P2.54mm_Vertical, symbol Connector:Conn_01x10_Socket
- removed J9: Conn_01x06_Socket, Connector_PinHeader_2.54mm:PinHeader_1x06_P2.54mm_Vertical, symbol Connector:Conn_01x06_Socket
- added A1: Arduino_Mega2560_R3_Shield, sparkfun-electromech:Arduino_Mega2560_R3_K3NG, symbol PCM_arduino-library:Arduino_Mega2560_R3_Shield
Connections:
- net 5V: now also A1.5V1 (5V)
- net AzimuthV: now also J7.1 (Pin_1); no longer J7.2 (Pin_2)
- net DOWN: now also A1.D46
- net ElevationV: now also J7.2 (Pin_2); no longer J7.1 (Pin_1)
- net GND: now also A1.GND1 (GND), A1.GND2 (GND), A1.GND3 (GND), A1.GND4 (SPI_GND), A1.GND5 (GND), A1.GND6 (GND)
- net IPRO1: now also A1.A2
- net IPRO2: now also A1.A3
- net RotateCCW: now also A1.D6
- net RotateCW: now also A1.D7
- net RotateDown: now also A1.D8
- net RotateUP: now also A1.D5
- net SCL: now also A1.SCL
- net SDA: now also A1.SDA
- net Turn CCW: now also A1.D44
- net Turn CW: now also A1.D43
- net UP: now also A1.D45
- net Vref: now also A1.3V3 (3.3V)
- net at J6.7 (Pin_7): now also A1.D47
- net at R1.2: now also A1.A1
- net at R2.2: now also A1.A0
- net ACD0: no longer names the net of J7.6 (Pin_6)
- no-connect marks 12 -> 70
Other:
- note added: "CONNECTIONS TO ARDUINO MEGA 2560"
- note removed: "ANALOG INPUTS ARDUINO"
- note removed: "AREF"
- note removed: "CONNECTIONS TO ARDUINO UNO"
- note removed: "D0/RX"
- note removed: "D1/TX"
- note removed: "D10"
- note removed: "D11"
- note removed: "D12"
- note removed: "D13"
- note removed: "D14"
- note removed: "D15"
- note removed: "D16"
- note removed: "D17"
- note removed: "D18"
- note removed: "D19"
- note removed: "D2"
- note removed: "D3"
- note removed: "D4"
- note removed: "D5"
- note removed: "D6"
- note removed: "D7"
- note removed: "D8"
- note removed: "D9"
- note removed: "GND"
- note removed: "GPIO"
- note removed: "I2C and other pins"
- note removed: "SLA"
- note removed: "SLC"
- note removed: "VREF,5V AND GND"
- moved on the sheet: C1, C2, C3, C4, J14, J2, J3, J4, J6, J7, R1, R2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
