File: K3NG-rotator-shield.kicad_sch (KiCad schematic)
At the start: 18 parts, among them J14 Conn_01x01_Pin, J15 Conn_01x01_Pin, J2 Conn_01x04_Socket, J3 Conn_01x02_Pin, J4 Conn_01x04_Socket, J6 Conn_01x07_Socket, J7 Conn_01x06_Socket, U1 DRV8251ADDAR, U2 DRV8251ADDAR

Commit message: Add files via upload
Other:
- note added: "A PCB with dual DRV8251A and connections to Arduino Mega 2560"
- note removed: "A PCB with dual DRV8251A and connections to Arduino Uno"
Changed lines of the file:
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@@
 		)
 	)
-	(text "A PCB with dual DRV8251A and connections to Arduino Uno"
+	(text "A PCB with dual DRV8251A and connections to Arduino Mega 2560"
 		(exclude_from_sim no)
 		(at 209.296 169.418 0)

Commit message: Add files via upload
Parts:
- J3: footprint Connector_PinHeader_2.54mm:PinHeader_1x02_P2.54mm_Vertical -> Connector_Wire:SolderWire-1.5sqmm_1x02_P6mm_D1.7mm_OD3mm
- R1, R2, R3, R4: footprint Resistor_THT:R_Axial_DIN0204_L3.6mm_D1.6mm_P5.08mm_Vertical -> Resistor_THT:R_Axial_DIN0204_L3.6mm_D1.6mm_P5.08mm_Horizontal
Connections:
- net GND: no longer A1.GND4 (SPI_GND)
- no-connect marks 70 -> 73
Changed lines of the file:
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@@
 	)
 	(no_connect
+		(at 217.17 24.13)
+	)
+	(no_connect
 		(at 177.8 109.22)
 	)
@@
 	)
 	(no_connect
+		(at 177.8 81.28)
+	)
+	(no_connect
 		(at 243.84 76.2)
 	)
@@
 	)
 	(no_connect
+		(at 177.8 78.74)
+	)
+	(no_connect
 		(at 177.8 50.8)
 	)
@@
 	(wire
 		(pts
-			(xy 217.17 24.13) (xy 223.52 24.13)
-		)
-		(stroke
-			(width 0)
-			(type default)
-		)
-	)
-	(wire
-		(pts
 			(xy 152.4 185.42) (xy 163.83 185.42)
 		)
@@
 			)
 		)
-		(property "Footprint" "Connector_PinHeader_2.54mm:PinHeader_1x02_P2.54mm_Vertical"
+		(property "Footprint" "Connector_Wire:SolderWire-1.5sqmm_1x02_P6mm_D1.7mm_OD3mm"
 			(at 38.1 30.48 0)
 			(effects
@@
 			)
 		)
-		(property "Footprint" "Resistor_THT:R_Axial_DIN0204_L3.6mm_D1.6mm_P5.08mm_Vertical"
+		(property "Footprint" "Resistor_THT:R_Axial_DIN0204_L3.6mm_D1.6mm_P5.08mm_Horizontal"
 			(at 38.862 88.9 90)
 			(effects
@@
 			)
 		)
-		(property "Footprint" "Resistor_THT:R_Axial_DIN0204_L3.6mm_D1.6mm_P5.08mm_Vertical"
+		(property "Footprint" "Resistor_THT:R_Axial_DIN0204_L3.6mm_D1.6mm_P5.08mm_Horizontal"
 			(at 165.1 72.898 90)
 			(effects
@@
 	)
 	(symbol
-		(lib_id "power:GND")
-		(at 223.52 24.13 0)
-		(unit 1)
-		(exclude_from_sim no)
-		(in_bom yes)
-		(on_board yes)
-		(dnp no)
-		(property "Reference" "#PWR015"
-			(at 223.52 30.48 0)
-			(effects
-				(font
-					(size 1.27 1.27)
-				)
-				(hide yes)
-			)
-		)
-		(property "Value" "GND"
-			(at 223.52 29.21 0)
-			(effects
-				(font
-					(size 1.27 1.27)
-				)
-			)
-		)
-		(property "Footprint" ""
-			(at 223.52 24.13 0)
-			(effects
-				(font
-					(size 1.27 1.27)
-				)
-				(hide yes)
-			)
-		)
-		(property "Datasheet" ""
-			(at 223.52 24.13 0)
-			(effects
-				(font
-					(size 1.27 1.27)
-				)
-				(hide yes)
-			)
-		)
-		(property "Description" "Power symbol creates a global label with name \"GND\" , ground"
-			(at 223.52 24.13 0)
-			(effects
-				(font
-					(size 1.27 1.27)
-				)
-				(hide yes)
-			)
-		)
-		(pin "1"
-		)
-		(instances
-			(project "K3NG-rotator-shield"
-				(path "/43396cf7-6229-4c16-b35b-9e1dd4c3617f"
-					(reference "#PWR015")
-					(unit 1)
-				)
-			)
-		)
-	)
-	(symbol
 		(lib_id "Device:C")
 		(at 143.51 77.47 0)
@@
 			)
 		)
-		(property "Footprint" "Resistor_THT:R_Axial_DIN0204_L3.6mm_D1.6mm_P5.08mm_Vertical"
+		(property "Footprint" "Resistor_THT:R_Axial_DIN0204_L3.6mm_D1.6mm_P5.08mm_Horizontal"
 			(at 165.1 69.088 90)
 			(effects
@@
 			)
 		)
-		(property "Footprint" "Resistor_THT:R_Axial_DIN0204_L3.6mm_D1.6mm_P5.08mm_Vertical"
+		(property "Footprint" "Resistor_THT:R_Axial_DIN0204_L3.6mm_D1.6mm_P5.08mm_Horizontal"
 			(at 40.132 132.08 90)
 			(effects

Commit message: Add files via upload
Parts:
- C1, C2, C3: mfr (none) -> K104K10X7RF5UH5
- C4: mfr (none) -> RNU1H470MDN1PH
- J2, J4: mfr (none) -> 1725672
- J6: Mfr (none) -> 1725708; mfr (none) -> 1725708
- J7: Mfr (none) -> 1725698; mfr (none) -> 1725698
- R1, R2: mfr (none) -> YR1B1K0CC
- R3, R4: mfr (none) -> MFR-25FBF52-1K3
Changed lines of the file:
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@@
 	(text "A PCB with dual DRV8251A and connections to Arduino Mega 2560"
 		(exclude_from_sim no)
-		(at 209.296 169.418 0)
+		(at 211.836 169.418 0)
 		(effects
 			(font
@@
 			)
 		)
+		(property "Mfr" "1725708"
+			(at 273.05 121.92 0)
+			(effects
+				(font
+					(size 1.27 1.27)
+				)
+				(hide yes)
+			)
+		)
+		(property "mfr" "1725708"
+			(at 273.05 121.92 0)
+			(effects
+				(font
+					(size 1.27 1.27)
+				)
+				(hide yes)
+			)
+		)
 		(pin "6"
 		)
@@
 			)
 		)
+		(property "mfr" "  RNU1H470MDN1PH"
+			(at 82.55 34.29 0)
+			(effects
+				(font
+					(size 1.27 1.27)
+				)
+				(hide yes)
+			)
+		)
 		(pin "1"
 		)
@@
 			)
 		)
+		(property "mfr" "  1725672"
+			(at 142.24 60.96 0)
+			(effects
+				(font
+					(size 1.27 1.27)
+				)
+				(hide yes)
+			)
+		)
 		(pin "4"
 		)
@@
 			)
 		)
+		(property "mfr" "  MFR-25FBF52-1K3"
+			(at 40.64 88.9 0)
+			(effects
+				(font
+					(size 1.27 1.27)
+				)
+				(hide yes)
+			)
+		)
 		(pin "2"
 		)
@@
 			)
 		)
+		(property "mfr" "  YR1B1K0CC"
+			(at 165.1 71.12 90)
+			(effects
+				(font
+					(size 1.27 1.27)
+				)
+				(hide yes)
+			)
+		)
 		(pin "2"
 		)
@@
 			)
 		)
+		(property "mfr" "K104K10X7RF5UH5"
+			(at 143.51 77.47 0)
+			(effects
+				(font
+					(size 1.27 1.27)
+				)
+				(hide yes)
+			)
+		)
 		(pin "1"
 		)
@@
 			)
 		)
+		(property "mfr" "  YR1B1K0CC"
+			(at 165.1 67.31 90)
+			(effects
+				(font
+					(size 1.27 1.27)
+				)
+				(hide yes)
+			)
+		)
 		(pin "2"
 		)
@@
 			)
 		)
+		(property "mfr" "K104K10X7RF5UH5"
+			(at 156.21 77.47 0)
+			(effects
+				(font
+					(size 1.27 1.27)
+				)
+				(hide yes)
+			)
+		)
 		(pin "1"
 		)
@@
 			)
 		)
+		(property "mfr" "  1725672"
+			(at 46.99 64.77 0)
+			(effects
+				(font
+					(size 1.27 1.27)
+				)
+				(hide yes)
+			)
+		)
 		(pin "3"
 		)
@@
 			)
 		)
+		(property "Mfr" "  1725698"
+			(at 132.08 72.39 0)
+			(effects
+				(font
+					(size 1.27 1.27)
+				)
+				(hide yes)
+			)
+		)
+		(property "mfr" "  1725698"
+			(at 132.08 72.39 0)
+			(effects
+				(font
+					(size 1.27 1.27)
+				)
+				(hide yes)
+			)
+		)
 		(pin "5"
 		)
@@
 			)
 		)
+		(property "mfr" "  MFR-25FBF52-1K3"
+			(at 41.91 132.08 0)
+			(effects
+				(font
+					(size 1.27 1.27)
+				)
+				(hide yes)
+			)
+		)
 		(pin "2"
 		)
@@
 			(at 69.85 34.29 0)
 			(effects
+				(font
+					(size 1.27 1.27)
+				)
+				(hide yes)
+			)
+		)
+		(property "mfr" "K104K10X7RF5UH5"
+			(at 69.85 34.29 0)
+			(effects
